Commit message: Account for gripper in the end effector link

File: drake/examples/kuka_iiwa_arm/models/iiwa14/iiwa14_simplified_collision.urdf (robot description, URDF)
Before this commit: robot iiwa14, 11 links, 10 joints
Joints:
- joint tool0_joint: origin xyz=0 0 0.045 rpy=0 -1.57079632679 0 -> xyz=0 0 0.220 rpy=0 -1.57079632679 -0.3922699

Commit message: turn down some joint limits and play with constraints

File: drake/examples/kuka_iiwa_arm/models/iiwa14/iiwa14_simplified_collision.urdf (robot description, URDF)
Before this commit: robot iiwa14, 11 links, 10 joints
Joints:
- joint iiwa_joint_1: limit lower=-2.96705972839 upper=2.96705972839 effort=300 velocity=10 -> lower=-2.8797933 upper=2.8797933 effort=300 velocity=10
- joint iiwa_joint_2: limit lower=-2.09439510239 upper=2.09439510239 effort=300 velocity=10 -> lower=-2.0071286 upper=2.0071286 effort=300 velocity=10
- joint iiwa_joint_4: limit lower=-2.09439510239 upper=2.09439510239 effort=300 velocity=10 -> lower=-2.0071286 upper=2.0071286 effort=300 velocity=10
- joint iiwa_joint_6: limit lower=-2.09439510239 upper=2.09439510239 effort=300 velocity=10 -> lower=-2.0071286 upper=2.0071286 effort=300 velocity=10
