Commit message: Jaco simulation!

File: manipulation/models/jaco_description/urdf/j2s7s300.urdf (robot description, URDF)
Before this commit: robot j2s7s300, 16 links, 15 joints
Links:
- link j2s7s300_link_base: geometry visual mesh filename=../meshes/base.obj

Commit message: Checkpoint again.  Something happens, but the resulting simulated motion doesn't make a hell of a lot of sense.  Sim error or planning error?  Who knows!

File: manipulation/models/jaco_description/urdf/j2s7s300.urdf (robot description, URDF)
Before this commit: robot j2s7s300, 16 links, 15 joints
Links:
- link base: geometry visual box size=0 0 0
- link j2s7s300_link_1: geometry visual mesh filename=../meshes/ring_big.obj; visual mesh filename=../meshes/shoulder.obj
- link j2s7s300_link_2: geometry visual mesh filename=../meshes/arm_half_1.obj; visual mesh filename=../meshes/ring_big.obj

Commit message: use fingered urdf

File: manipulation/models/jaco_description/urdf/j2s7s300.urdf (robot description, URDF)
Before this commit: robot j2s7s300, 16 links, 15 joints
Joints:
- joint j2s7s300_joint_end_effector: origin xyz=0 0 -0.1600 rpy=3.14159265359 0 0 -> xyz=0 0 -0.1600 rpy=1.57079632679 1.57079632679 1.57079632679

Commit message: Tweaks from running the demo on hardware

File: manipulation/models/jaco_description/urdf/j2s7s300.urdf (robot description, URDF)
Before this commit: robot j2s7s300, 16 links, 15 joints
Joints:
- joint j2s7s300_joint_base: origin xyz=0 0 0 rpy=0 0 0 -> xyz=0 0 0 rpy=0 0 1.57079632679
